File: watch-dk/MCU.kicad_sch (KiCad schematic)
At the start: 41 parts, among them IC601 FAN5622SX, IC602 USBLC6-2P6, IC603 MX25U51245GZ4I00, IC604 NTS0104GU12, J601 Jumper, J602 Jumper, J603 Jumper, J604 Jumper, M601 NORA-B106, X601 DEBUG, X602 Current, X603 Device, X604 UART, X605 GPIO, X606 Current, X607 IO Current, X608 Display, X609 Touch Current, X610 LED Current

Commit message: Fix wrong part number for SWD connector, fix missing footprint for RTC level shifter, cosmetic changes
Parts:
- X601: manf# 623310235521 -> 62101021021; mouser# 710-623310235521 -> 710-62101021021
Changed lines of the file:
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@@
 			)
 		)
-		(property "manf#" "623310235521"
+		(property "manf#" "62101021021"
 			(at 41.91 255.27 0)
 			(effects
@@
 			)
 		)
-		(property "mouser#" "710-623310235521"
+		(property "mouser#" "710-62101021021"
 			(at 41.91 255.27 0)
 			(effects
